File: X15_Power_Plate.sch (EAGLE design)
At the start: 26 parts

Commit message: power conversion layout finished
Parts:
- removed U$1: CONN_DISTRIBUTION_TO_CONVERSION, X15_Brickstribution:CONN_DISTRIBUTION_TO_CONVERSION
- added C10: 10uF, SparkFun-Capacitors:4.7PF-0603-50V-5%
- added C11: 22uF, SparkFun-Capacitors:4.7PF-0603-50V-5%
- added CIN1: 180uF, X15-Conversion-Parts-Library:EEEFKE181XSP
- added CIN2, CIN3: 4.7uF, SparkFun-Capacitors:4.7UF0603
- added COUT1, COUT2, COUT3: 150uF, X15-Conversion-Parts-Library:C-TANTALUM(10UF_150UF)
- added D10: BLUE, SparkFun-LED:LED-BLUE0603
- added D11: WHITE, SparkFun-LED:LED-WHITE0603
- added D13: GREEN, SparkFun-LED:LED-GREEN0603
- added L1: 15uH, X15-Conversion-Parts-Library:HCMA1305
- added R2: 1k, SparkFun-Resistors:2.0KOHM-0603-1/10W-5%
- added R3: 3.32k, SparkFun-Resistors:2.0KOHM-0603-1/10W-5%
- added R4: 100, SparkFun-Resistors:100OHM-0603-1/4W-5%
- added R7: 470, SparkFun-Resistors:470OHM-0603-1/10W-1%
- added R8: 20, SparkFun-Resistors:20OHM-0603-1/10W-1%
- added RADJ: 12.4k, SparkFun-Resistors:2.0KOHM-0603-1/10W-5%
- added U$6: BUCK,LM2679SX-ADJ, X15-Conversion-Parts-Library:BUCK,LM2679SX-ADJ
- added U$7: CDBG520-G, X15-Conversion-Parts-Library:CDBG520-G
- added U1: LINEAR,AZ1117CR-3.3TRG1DIODES_AZ1117CH-3.3TRG1_0_0, X15-Conversion-Parts-Library:LINEAR,AZ1117CR-3.3TRG1DIODES_AZ1117CH-3.3TRG1_0_0
Connections:
- new net N$12: D11.A, R8.2
- new net N$2: R2.1, R3.1, U$6.FB
- new net N$3: D13.A, R7.2
- new net N$4: CIN3.2, L1.1, U$6.SWITCH, U$7.1
- new net N$5: CIN3.1, U$6.BOOST
- new net N$8: RADJ.2, U$6.CRADJ
- new net N$9: D10.A, R4.2
- net +12V: now also CIN1.1, CIN2.1, R7.1, U$6.VIN; no longer U$1.VIN+, U$1.VIN-
- net +3.3V: now also C11.1, R8.1, U1.OUPUT; no longer U$1.VOUT+_3
- net +5V: now also C10.1, COUT1.+, COUT2.+, COUT3.+, L1.2, R3.2, R4.1, U1.INPUT; no longer U$1.VOUT+_5
- net 12V_GND: now also C10.2, C11.2, CIN1.2, CIN2.2, COUT1.-, COUT2.-, COUT3.-, D10.C, D11.C, D13.C, R2.2, RADJ.1, U$6.GND, U$7.2, U1.GND; no longer U$1.VOUT-
- net 48V_GND: now also U$2.RMCONT
Other:
- note added: "Power Conversion Board Components"
- note added: "Test Voltage LEDs"
- note removed: "Connector to conversion Board"
- moved on the sheet: +12V_TEST, +3.3V_TEST, +5V_TEST, 12V-5V-3.3V_GND, 48V_GND_TEST, 48V_TEST, D1, PI_SHIELD_CONN1, R1, U$3
